Commit message: Fixes multi-robot sim.

File: src/follow_path/fetch_description_pkg/robots/fetch.gazebo.xacro (robot description, xacro)
@@ -1,4 +1,4 @@
 <robot xmlns:xacro="http://www.ros.org/wiki/xacro" name="fetch" >
-  <xacro:include filename="$(find fetch_description)/robots/fetch.urdf" />
+  <xacro:include filename="$(find fetch_description_pkg)/robots/fetch.urdf" />
   <!-- Add four casters to the base -->
   <xacro:macro name="caster" params="prefix joint_x joint_y">

File: src/follow_path/turtlebot3_description_pkg/urdf/turtlebot3_burger.urdf.xacro (robot description, xacro)
@@ -1,6 +1,6 @@
 <?xml version="1.0" ?>
 <robot name="turtlebot3_burger" xmlns:xacro="http://ros.org/wiki/xacro">
-  <xacro:include filename="$(find turtlebot3_description)/urdf/common_properties.xacro"/>
-  <xacro:include filename="$(find turtlebot3_description)/urdf/turtlebot3_burger.gazebo.xacro"/>
+  <xacro:include filename="$(find turtlebot3_description_pkg)/urdf/common_properties.xacro"/>
+  <xacro:include filename="$(find turtlebot3_description_pkg)/urdf/turtlebot3_burger.gazebo.xacro"/>
   <link name="base_footprint"/>
   <joint name="base_joint" type="fixed">
@@ -13,5 +13,5 @@
       <origin xyz="-0.032 0 0.0" rpy="0 0 0"/>
       <geometry>
-        <mesh filename="package://turtlebot3_description/meshes/bases/burger_base.stl" scale="0.001 0.001 0.001"/>
+        <mesh filename="package://turtlebot3_description_pkg/meshes/bases/burger_base.stl" scale="0.001 0.001 0.001"/>
       </geometry>
       <material name="light_black"/>
@@ -41,5 +41,5 @@
       <origin xyz="0 0 0" rpy="1.57 0 0"/>
       <geometry>
-        <mesh filename="package://turtlebot3_description/meshes/wheels/left_tire.stl" scale="0.001 0.001 0.001"/>
+        <mesh filename="package://turtlebot3_description_pkg/meshes/wheels/left_tire.stl" scale="0.001 0.001 0.001"/>
       </geometry>
       <material name="dark"/>
@@ -69,5 +69,5 @@
       <origin xyz="0 0 0" rpy="1.57 0 0"/>
       <geometry>
-        <mesh filename="package://turtlebot3_description/meshes/wheels/right_tire.stl" scale="0.001 0.001 0.001"/>
+        <mesh filename="package://turtlebot3_description_pkg/meshes/wheels/right_tire.stl" scale="0.001 0.001 0.001"/>
       </geometry>
       <material name="dark"/>
@@ -134,5 +134,5 @@
       <origin xyz="0 0 0.0" rpy="0 0 0"/>
       <geometry>
-        <mesh filename="package://turtlebot3_description/meshes/sensors/lds.stl" scale="0.001 0.001 0.001"/>
+        <mesh filename="package://turtlebot3_description_pkg/meshes/sensors/lds.stl" scale="0.001 0.001 0.001"/>
       </geometry>
       <material name="dark"/>
